File: pcb/FPGA_IO.sch (KiCad schematic (older format))
At the start: 9 parts, among them J2 JSHORTNORMAL, J3 JSHORTNORMAL, U4 iCE40-HX8K-CT256, U7 OSC

Commit message: Generated the gerbers and submitted them. * Added some 3D models.
Parts:
- JP1, JP5: footprint open-project:S_JUMPER_2 -> XESS:S_JUMPER_2
- renumbered J2 to SH5, J3 to SH6
Changed lines of the file:
@@
 1E 25 49 2A DA F6 C4 5C B7 0C C3 B9 A4 0A 98 09 FC 0D B0 92 CD 57 CD 1F 06 4E 04 26 A7 75 27 49
 52 39 26 13 73 DE C3 6C BE 70 B5 12 F8 16 86 73 8D C3 FF 03 63 F8 EE 2E BE 9A 04 B1 00 00 00 00
-49 45 4E 44 AE 42 60 82 8C
+49 45 4E 44 AE 42 60 82 40
 EndData
 $EndBitmap
@@
 F 0 "JP5" H 8800 1750 50  0000 C CNN
 F 1 "JUMPER" H 8800 1720 50  0001 C CNN
-F 2 "open-project:S_JUMPER_2" H 8800 1800 60  0001 C CNN
+F 2 "XESS:S_JUMPER_2" H 8800 1800 60  0001 C CNN
 F 3 "" H 8800 1800 60  0000 C CNN
 	1    8800 1800
@@
 F 0 "JP1" H 8800 1100 50  0000 C CNN
 F 1 "JUMPER" H 8800 1070 50  0001 C CNN
-F 2 "open-project:S_JUMPER_2" H 8800 1150 60  0001 C CNN
+F 2 "XESS:S_JUMPER_2" H 8800 1150 60  0001 C CNN
 F 3 "" H 8800 1150 60  0000 C CNN
 	1    8800 1150
@@
 P 8850 1300
 AR Path="/55F913D4" Ref="J?"  Part="1"
-AR Path="/55DF5F27/55E883EA/55F049F2/55F913D4" Ref="J2"  Part="1"
-F 0 "J2" H 8850 1200 50  0001 L BNN
+AR Path="/55DF5F27/55E883EA/55F049F2/55F913D4" Ref="SH5"  Part="1"
+F 0 "SH5" H 8850 1200 50  0001 L BNN
 F 1 "JSHORTNORMAL" H 8750 1200 50  0001 L BNN
 F 2 "XESS:xess-JSHORT" H 8850 1450 50  0001 C CNN
@@
 P 8850 1950
 AR Path="/55F913E4" Ref="J?"  Part="1"
-AR Path="/55DF5F27/55E883EA/55F049F2/55F913E4" Ref="J3"  Part="1"
-F 0 "J3" H 8850 1850 50  0001 L BNN
+AR Path="/55DF5F27/55E883EA/55F049F2/55F913E4" Ref="SH6"  Part="1"
+F 0 "SH6" H 8850 1850 50  0001 L BNN
 F 1 "JSHORTNORMAL" H 8750 1850 50  0001 L BNN
 F 2 "XESS:xess-JSHORT" H 8850 2100 50  0001 C CNN

Commit message: Added manufacturer part numbers to the schematic.
Parts:
- R7: symbol R_Small -> R; manf# (none) -> RC0603JR-07100RL
- RN4: value 10K -> 4.7K
- U7: value OSC -> 100 MHz Osc
Other:
- moved on the sheet: R7
Changed lines of the file:
@@
 1E 25 49 2A DA F6 C4 5C B7 0C C3 B9 A4 0A 98 09 FC 0D B0 92 CD 57 CD 1F 06 4E 04 26 A7 75 27 49
 52 39 26 13 73 DE C3 6C BE 70 B5 12 F8 16 86 73 8D C3 FF 03 63 F8 EE 2E BE 9A 04 B1 00 00 00 00
-49 45 4E 44 AE 42 60 82 40
+49 45 4E 44 AE 42 60 82 13
 EndData
 $EndBitmap
@@
 P 3450 7050
 F 0 "U7" H 3650 7300 60  0000 L CNN
-F 1 "OSC" H 3650 7200 60  0000 L CNN
+F 1 "100 MHz Osc" H 3650 7200 60  0000 L CNN
 F 2 "XESS:2.5x3.2" H 3450 7050 50  0001 C CNN
 F 3 "" H 3450 7050 50  0000 C CNN
@@
 P 9600 1300
 F 0 "RN4" H 9750 1200 50  0000 C CNN
-F 1 "10K" H 9750 1300 50  0000 C CNN
+F 1 "4.7K" H 9750 1300 50  0000 C CNN
 F 2 "XESS:CTS_742C043" H 9600 1300 50  0001 C CNN
 F 3 "" H 9600 1300 50  0000 C CNN
@@
 P 9800 1300
 F 0 "RN4" H 9950 1200 50  0000 C CNN
-F 1 "10K" H 9950 1300 50  0000 C CNN
+F 1 "4.7K" H 9950 1300 50  0000 C CNN
 F 2 "XESS:CTS_742C043" H 9800 1300 50  0001 C CNN
 F 3 "" H 9800 1300 50  0000 C CNN
@@
 	1    0    0    -1
 $EndComp
-Text GLabel 8200 1500 0    50   Input ~ 0
+Text GLabel 8150 1500 0    50   Input ~ 0
 GND
 $Comp
@@
 USER_CLK
 Wire Wire Line
-	9900 1500 9100 1500
+	9100 1500 9900 1500
 Wire Wire Line
 	9600 1300 9600 1500
@@
 Connection ~ 9800 1400
 $Comp
-L R_Small R7
+L R R7
 U 1 1 55FA4B25
-P 8350 1500
-F 0 "R7" V 8250 1450 50  0000 L CNN
-F 1 "100" V 8350 1500 40  0000 C CNN
-F 2 "Resistors_SMD:R_0603" H 8350 1500 60  0001 C CNN
-F 3 "" H 8350 1500 60  0000 C CNN
-	1    8350 1500
+P 8300 1500
+F 0 "R7" V 8200 1450 50  0000 L CNN
+F 1 "100" V 8300 1500 40  0000 C CNN
+F 2 "Resistors_SMD:R_0603" H 8300 1500 60  0001 C CNN
+F 3 "" H 8300 1500 60  0000 C CNN
+F 4 "RC0603JR-07100RL" V 8300 1500 60  0001 C CNN "manf#"
+	1    8300 1500
 	0    -1   -1   0
 $EndComp
 Wire Wire Line
-	8200 1500 8250 1500
-Wire Wire Line
 	8450 1500 8500 1500
