File: pcb/FPGA_IO.sch (KiCad schematic (older format))
At the start: 9 parts, among them U4 iCE40-HX8K-CT256, U7 100 MHz Osc

Commit message: Added assembly order field to schematic.
Parts:
- R7: assembly_order (none) -> 38
- RESET1: assembly_order (none) -> 71
- RN4: assembly_order (none) -> 58
- U4: assembly_order (none) -> 1; manf# (none) -> ICE40HX8K-CT256
- U7: assembly_order (none) -> 2

Commit message: Assembly order field stopped propagation of part numbers, so I added them to each part using kifield.
Parts:
- RESET1: manf# (none) -> RS-282G05A3-SM RT
- RN4: manf# (none) -> 742C043472JP
Changed lines of the file:
@@
 F 3 "" H 9600 1300 50 0000 C CNN
 F 4 "58" H 0 0 50 0001 C CNN "assembly_order"
+F 5 "742C043472JP" H 0 0 50 0001 C CNN "manf#"
 	1    9600 1300
 	0    -1   -1   0
@@
 F 3 "" H 9800 1300 50 0000 C CNN
 F 4 "58" H 0 0 50 0001 C CNN "assembly_order"
+F 5 "742C043472JP" H 0 0 50 0001 C CNN "manf#"
 	2    9800 1300
 	0    -1   -1   0
@@
 F 3 "" H 8800 1500 60 0000 C CNN
 F 4 "71" H 0 0 50 0001 C CNN "assembly_order"
+F 5 "RS-282G05A3-SM RT" H 0 0 50 0001 C CNN "manf#"
 	1    8800 1500
 	1    0    0    -1

Commit message: CAT Board before new KiCad V5 schematic lib change.
Parts:
- JP1, JP5: symbol JUMPER -> JUMPER-RESCUE-CAT

Commit message: Works with KiCad V5.
Parts:
- JP1, JP5: symbol JUMPER-RESCUE-CAT -> CAT-rescue:JUMPER-RESCUE-CAT
- R7: symbol R -> device:R
- RESET1: symbol SW_PUSH -> CAT-rescue:SW_PUSH
- RN4: symbol RN2 -> XESS:RN2
- SH5, SH6: symbol JSHORTNORMAL -> XESS:JSHORTNORMAL
- U4: symbol iCE40-HX8K-CT256 -> Lattice-iCE:iCE40-HX8K-CT256
- U7: symbol OSC -> XESS:OSC
Changed lines of the file:
@@
-EESchema Schematic File Version 2
-LIBS:CAT-rescue
-LIBS:power
-LIBS:device
-LIBS:transistors
-LIBS:conn
-LIBS:linear
-LIBS:regul
-LIBS:74xx
-LIBS:cmos4000
-LIBS:adc-dac
-LIBS:memory
-LIBS:xilinx
-LIBS:microcontrollers
-LIBS:dsp
-LIBS:microchip
-LIBS:analog_switches
-LIBS:motorola
-LIBS:texas
-LIBS:intel
-LIBS:audio
-LIBS:interface
-LIBS:digital-audio
-LIBS:philips
-LIBS:display
-LIBS:cypress
-LIBS:siliconi
-LIBS:opto
-LIBS:atmel
-LIBS:contrib
-LIBS:valves
-LIBS:xess
-LIBS:Cypress_PSoC
-LIBS:Cypress_cy8c5xlp
-LIBS:Lattice_iCE_FPGA
-LIBS:xilinx7
-LIBS:xilinx6v
-LIBS:xilinx6s
-LIBS:xula
-LIBS:espressif-xess
+EESchema Schematic File Version 4
 LIBS:CAT-cache
 EELAYER 26 0
@@
 $EndDescr
 $Comp
-L iCE40-HX8K-CT256 U?
+L Lattice-iCE:iCE40-HX8K-CT256 U?
 U 2 1 55F04D7F
 P 1400 900
@@
 $EndComp
 $Comp
-L iCE40-HX8K-CT256 U?
+L Lattice-iCE:iCE40-HX8K-CT256 U?
 U 3 1 55F04D86
 P 3400 900
@@
 $EndComp
 $Comp
-L iCE40-HX8K-CT256 U?
+L Lattice-iCE:iCE40-HX8K-CT256 U?
 U 4 1 55F04D8D
 P 9900 1400
@@
 $EndComp
 $Comp
-L iCE40-HX8K-CT256 U?
+L Lattice-iCE:iCE40-HX8K-CT256 U?
 U 5 1 55F04D94
 P 5400 900
@@
 $EndComp
 $Comp
-L OSC U7
+L XESS:OSC U7
 U 1 1 55F1B092
 P 3450 7050
@@
 $EndComp
 $Comp
-L RN2 RN4
+L XESS:RN2 RN4
 U 1 1 55F1B0FB
 P 9600 1300
@@
 $EndComp
 $Comp
-L RN2 RN4
+L XESS:RN2 RN4
 U 2 1 55F1B188
 P 9800 1300
@@
 $EndComp
 $Comp
-L SW_PUSH RESET1
+L CAT-rescue:SW_PUSH RESET1
 U 1 1 55F43F78
 P 8800 1500
@@
 $EndComp
 $Comp
-L JUMPER-RESCUE-CAT JP5
+L CAT-rescue:JUMPER-RESCUE-CAT JP5
 U 1 1 55F44072
 P 8800 1800
@@
 $EndComp
 $Comp
-L JUMPER-RESCUE-CAT JP1
+L CAT-rescue:JUMPER-RESCUE-CAT JP1
 U 1 1 55F4436F
 P 8800 1150
@@
 $EndComp
 $Comp
-L JSHORTNORMAL J?
+L XESS:JSHORTNORMAL J?
 U 1 1 55F913D4
 P 8850 1300
@@
 $EndComp
 $Comp
-L JSHORTNORMAL J?
+L XESS:JSHORTNORMAL J?
 U 1 1 55F913E4
 P 8850 1950
@@
 $EndComp
 $Comp
-L R R7
+L device:R R7
 U 1 1 55FA4B25
 P 8300 1500
@@
 GR3-IO2
 Wire Wire Line
-	2900 3700 3400 3700
+	2900 3700 3000 3700
 Wire Wire Line
 	3400 3900 3000 3900
@@
 	3000 3900 3000 3700
 Wire Wire Line
-	9100 1500 9900 1500
+	9100 1500 9200 1500
 Wire Wire Line
 	9600 1300 9600 1500
@@
 	9200 1300 9200 1150
 Wire Wire Line
-	9100 1150 9400 1150
+	9100 1150 9200 1150
 Wire Wire Line
 	9400 1150 9400 1400
 Wire Wire Line
-	9400 1400 9900 1400
+	9400 1400 9800 1400
 Wire Wire Line
 	9800 1300 9800 1400
@@
 NoConn ~ 9900 6000
 NoConn ~ 9900 6100
+Wire Wire Line
+	3000 3700 3400 3700
+Wire Wire Line
+	9600 1500 9900 1500
+Wire Wire Line
+	9200 1500 9600 1500
+Wire Wire Line
+	9200 1150 9400 1150
+Wire Wire Line
+	9800 1400 9900 1400
 $EndSCHEMATC
