File: pcb/FPGA_PWR.sch (KiCad schematic (older format))
At the start: 37 parts, among them U4 iCE40-HX8K-CT256, U8 AZ1117EH-ADJ

Commit message: Added assembly order field to schematic.
Parts:
- C16: assembly_order (none) -> 19
- C17: assembly_order (none) -> 5
- C18: assembly_order (none) -> 29
- C19: assembly_order (none) -> 24
- C20: assembly_order (none) -> 18
- C21: assembly_order (none) -> 12
- C22: assembly_order (none) -> 28
- C23: assembly_order (none) -> 23
- C24: assembly_order (none) -> 17
- C25: assembly_order (none) -> 32
- C26: assembly_order (none) -> 30
- C27: assembly_order (none) -> 21
- C28: assembly_order (none) -> 16
- C29: assembly_order (none) -> 35
- C30: assembly_order (none) -> 26
- C31: assembly_order (none) -> 20
- C32: assembly_order (none) -> 27
- C33: assembly_order (none) -> 10
- C34: assembly_order (none) -> 6
- C35: assembly_order (none) -> 11
- C38: assembly_order (none) -> 22
- C39: assembly_order (none) -> 15
- C40: assembly_order (none) -> 9
- C41: assembly_order (none) -> 14
- C42: assembly_order (none) -> 7
- C43: assembly_order (none) -> 13
- C44: assembly_order (none) -> 4
- C45: assembly_order (none) -> 31
- C46: assembly_order (none) -> 3
- C6: assembly_order (none) -> 45
- D1: assembly_order (none) -> 34
- R1: assembly_order (none) -> 33
- R6: assembly_order (none) -> 8
- R8: assembly_order (none) -> 48
- R9: assembly_order (none) -> 47
- U4: assembly_order (none) -> 1
- U8: assembly_order (none) -> 51

Commit message: Assembly order field stopped propagation of part numbers, so I added them to each part using kifield.
Parts:
- C17, C18, C19, C24, C25, C26, C27, C34, C35, C40, C41, C42, C44, C45: manf# (none) -> GRM188R71C104KA01D
- C21, C22, C23, C28, C29, C30, C31, C38, C39: manf# (none) -> GRM188R71C105KE15D
- C32, C33, C6: manf# (none) -> GRM21BR61A106KE19L
- C46: manf# (none) -> GRM188R71H103KA01D
- R1, R6: manf# (none) -> RC0603JR-07100RL
Changed lines of the file:
@@
 F 3 "" H 4800 3850 60 0000 C CNN
 F 4 "17" H 0 0 50 0001 C CNN "assembly_order"
+F 5 "GRM188R71C104KA01D" H 0 0 50 0001 C CNN "manf#"
 	1    4800 3850
 	1    0    0    -1
@@
 F 3 "" H 5100 3850 60 0000 C CNN
 F 4 "16" H 0 0 50 0001 C CNN "assembly_order"
+F 5 "GRM188R71C105KE15D" H 0 0 50 0001 C CNN "manf#"
 	1    5100 3850
 	1    0    0    -1
@@
 F 3 "" H 4200 4450 60 0000 C CNN
 F 4 "5" H 0 0 50 0001 C CNN "assembly_order"
+F 5 "GRM188R71C104KA01D" H 0 0 50 0001 C CNN "manf#"
 	1    4200 4450
 	1    0    0    -1
@@
 F 3 "" H 4500 4450 60 0000 C CNN
 F 4 "12" H 0 0 50 0001 C CNN "assembly_order"
+F 5 "GRM188R71C105KE15D" H 0 0 50 0001 C CNN "manf#"
 	1    4500 4450
 	1    0    0    -1
@@
 F 3 "" H 4800 4450 60 0000 C CNN
 F 4 "32" H 0 0 50 0001 C CNN "assembly_order"
+F 5 "GRM188R71C104KA01D" H 0 0 50 0001 C CNN "manf#"
 	1    4800 4450
 	1    0    0    -1
@@
 F 3 "" H 5100 4450 60 0000 C CNN
 F 4 "35" H 0 0 50 0001 C CNN "assembly_order"
+F 5 "GRM188R71C105KE15D" H 0 0 50 0001 C CNN "manf#"
 	1    5100 4450
 	1    0    0    -1
@@
 F 3 "" H 4200 5050 60 0000 C CNN
 F 4 "29" H 0 0 50 0001 C CNN "assembly_order"
+F 5 "GRM188R71C104KA01D" H 0 0 50 0001 C CNN "manf#"
 	1    4200 5050
 	1    0    0    -1
@@
 F 3 "" H 4500 5050 60 0000 C CNN
 F 4 "28" H 0 0 50 0001 C CNN "assembly_order"
+F 5 "GRM188R71C105KE15D" H 0 0 50 0001 C CNN "manf#"
 	1    4500 5050
 	1    0    0    -1
@@
 F 3 "" H 4800 5050 60 0000 C CNN
 F 4 "30" H 0 0 50 0001 C CNN "assembly_order"
+F 5 "GRM188R71C104KA01D" H 0 0 50 0001 C CNN "manf#"
 	1    4800 5050
 	1    0    0    -1
@@
 F 3 "" H 5100 5050 60 0000 C CNN
 F 4 "26" H 0 0 50 0001 C CNN "assembly_order"
+F 5 "GRM188R71C105KE15D" H 0 0 50 0001 C CNN "manf#"
 	1    5100 5050
 	1    0    0    -1
@@
 F 3 "" H 4200 5650 60 0000 C CNN
 F 4 "24" H 0 0 50 0001 C CNN "assembly_order"
+F 5 "GRM188R71C104KA01D" H 0 0 50 0001 C CNN "manf#"
 	1    4200 5650
 	1    0    0    -1
@@
 F 3 "" H 4500 5650 60 0000 C CNN
 F 4 "23" H 0 0 50 0001 C CNN "assembly_order"
+F 5 "GRM188R71C105KE15D" H 0 0 50 0001 C CNN "manf#"
 	1    4500 5650
 	1    0    0    -1
@@
 F 3 "" H 4800 5650 60 0000 C CNN
 F 4 "21" H 0 0 50 0001 C CNN "assembly_order"
+F 5 "GRM188R71C104KA01D" H 0 0 50 0001 C CNN "manf#"
 	1    4800 5650
 	1    0    0    -1
@@
 F 3 "" H 5100 5650 60 0000 C CNN
 F 4 "20" H 0 0 50 0001 C CNN "assembly_order"
+F 5 "GRM188R71C105KE15D" H 0 0 50 0001 C CNN "manf#"
 	1    5100 5650
 	1    0    0    -1
@@
 F 3 "" H 5550 1850 60 0000 C CNN
 F 4 "6" H 0 0 50 0001 C CNN "assembly_order"
+F 5 "GRM188R71C104KA01D" H 0 0 50 0001 C CNN "manf#"
 	1    5550 1850
 	1    0    0    -1
@@
 F 3 "" H 5300 1850 60 0000 C CNN
 F 4 "27" H 0 0 50 0001 C CNN "assembly_order"
+F 5 "GRM21BR61A106KE19L" H 0 0 50 0001 C CNN "manf#"
 	1    5300 1850
 	1    0    0    -1
@@
 F 3 "" H 5550 2350 60 0000 C CNN
 F 4 "11" H 0 0 50 0001 C CNN "assembly_order"
+F 5 "GRM188R71C104KA01D" H 0 0 50 0001 C CNN "manf#"
 	1    5550 2350
 	1    0    0    -1
@@
 F 3 "" H 5300 2350 60 0000 C CNN
 F 4 "10" H 0 0 50 0001 C CNN "assembly_order"
+F 5 "GRM21BR61A106KE19L" H 0 0 50 0001 C CNN "manf#"
 	1    5300 2350
 	1    0    0    -1
@@
 F 3 "" H 6800 3850 60 0000 C CNN
 F 4 "22" H 0 0 50 0001 C CNN "assembly_order"
+F 5 "GRM188R71C105KE15D" H 0 0 50 0001 C CNN "manf#"
 	1    6800 3850
 	1    0    0    -1
@@
 F 3 "" H 7100 3850 60 0000 C CNN
 F 4 "9" H 0 0 50 0001 C CNN "assembly_order"
+F 5 "GRM188R71C104KA01D" H 0 0 50 0001 C CNN "manf#"
 	1    7100 3850
 	1    0    0    -1
@@
 F 3 "" H 7400 3850 60 0000 C CNN
 F 4 "7" H 0 0 50 0001 C CNN "assembly_order"
+F 5 "GRM188R71C104KA01D" H 0 0 50 0001 C CNN "manf#"
 	1    7400 3850
 	1    0    0    -1
@@
 F 3 "" H 7700 3850 60 0000 C CNN
 F 4 "4" H 0 0 50 0001 C CNN "assembly_order"
+F 5 "GRM188R71C104KA01D" H 0 0 50 0001 C CNN "manf#"
 	1    7700 3850
 	1    0    0    -1
@@
 F 3 "" H 8000 3850 60 0000 C CNN
 F 4 "31" H 0 0 50 0001 C CNN "assembly_order"
+F 5 "GRM188R71C104KA01D" H 0 0 50 0001 C CNN "manf#"
 	1    8000 3850
 	1    0    0    -1
@@
 F 3 "" H 8300 3850 60 0000 C CNN
 F 4 "3" H 0 0 50 0001 C CNN "assembly_order"
+F 5 "GRM188R71H103KA01D" H 0 0 50 0001 C CNN "manf#"
 	1    8300 3850
 	1    0    0    -1
@@
 F 3 "" H 6800 4450 60 0000 C CNN
 F 4 "15" H 0 0 50 0001 C CNN "assembly_order"
+F 5 "GRM188R71C105KE15D" H 0 0 50 0001 C CNN "manf#"
 	1    6800 4450
 	1    0    0    -1
@@
 F 3 "" H 7100 4450 60 0000 C CNN
 F 4 "14" H 0 0 50 0001 C CNN "assembly_order"
+F 5 "GRM188R71C104KA01D" H 0 0 50 0001 C CNN "manf#"
 	1    7100 4450
 	1    0    0    -1
@@
 F 3 "" H 5150 2000 30 0000 C CNN
 F 4 "33" H 0 0 50 0001 C CNN "assembly_order"
+F 5 "RC0603JR-07100RL" H 0 0 50 0001 C CNN "manf#"
 	1    5150 2000
 	0    1    1    0
@@
 F 3 "" H 5150 2500 30 0000 C CNN
 F 4 "8" H 0 0 50 0001 C CNN "assembly_order"
+F 5 "RC0603JR-07100RL" H 0 0 50 0001 C CNN "manf#"
 	1    5150 2500
 	0    1    1    0
@@
 F 3 "" H 3650 5650 60 0000 C CNN
 F 4 "45" H 0 0 50 0001 C CNN "assembly_order"
+F 5 "GRM21BR61A106KE19L" H 0 0 50 0001 C CNN "manf#"
 	1    3650 5650
 	1    0    0    -1

Commit message: Works with KiCad V5.
Parts:
- C16, C17, C18, C19, C20, C21, C22, C23, C24, C25, C26, C27, C28, C29, C30, C31, C32, C33, C34, C35, C38, C39, C40, C41, C42, C43, C44, C45, C46, C6: symbol C -> device:C
- D1: symbol D -> device:D
- R1, R6, R8, R9: symbol R -> device:R
- U4: symbol iCE40-HX8K-CT256 -> Lattice-iCE:iCE40-HX8K-CT256
- U8: symbol NCV1117 -> XESS:NCV1117
