File: pcb/Memory.sch (KiCad schematic (older format))
At the start: 8 parts, among them U5 16Mx16 SDRAM

Commit message: Added assembly order field to schematic.
Parts:
- C10: assembly_order (none) -> 36
- C11: assembly_order (none) -> 43
- C12: assembly_order (none) -> 42
- C13: assembly_order (none) -> 37
- C14: assembly_order (none) -> 40
- C8: assembly_order (none) -> 41
- C9: assembly_order (none) -> 39
- U5: assembly_order (none) -> 65

Commit message: Assembly order field stopped propagation of part numbers, so I added them to each part using kifield.
Parts:
- C10, C12, C14: manf# (none) -> GRM188R71C104KA01D
- C11, C13, C9: manf# (none) -> GRM188R71C105KE15D
Changed lines of the file:
@@
 F 3 "" H 6350 5750 60 0000 C CNN
 F 4 "42" H 0 0 50 0001 C CNN "assembly_order"
+F 5 "GRM188R71C104KA01D" H 0 0 50 0001 C CNN "manf#"
 	1    6350 5750
 	1    0    0    -1
@@
 F 3 "" H 6650 5750 60 0000 C CNN
 F 4 "37" H 0 0 50 0001 C CNN "assembly_order"
+F 5 "GRM188R71C105KE15D" H 0 0 50 0001 C CNN "manf#"
 	1    6650 5750
 	1    0    0    -1
@@
 F 3 "" H 6950 5750 60 0000 C CNN
 F 4 "40" H 0 0 50 0001 C CNN "assembly_order"
+F 5 "GRM188R71C104KA01D" H 0 0 50 0001 C CNN "manf#"
 	1    6950 5750
 	1    0    0    -1
@@
 F 3 "" H 5450 5750 60 0000 C CNN
 F 4 "39" H 0 0 50 0001 C CNN "assembly_order"
+F 5 "GRM188R71C105KE15D" H 0 0 50 0001 C CNN "manf#"
 	1    5450 5750
 	1    0    0    -1
@@
 F 3 "" H 5750 5750 60 0000 C CNN
 F 4 "36" H 0 0 50 0001 C CNN "assembly_order"
+F 5 "GRM188R71C104KA01D" H 0 0 50 0001 C CNN "manf#"
 	1    5750 5750
 	1    0    0    -1
@@
 F 3 "" H 6050 5750 60 0000 C CNN
 F 4 "43" H 0 0 50 0001 C CNN "assembly_order"
+F 5 "GRM188R71C105KE15D" H 0 0 50 0001 C CNN "manf#"
 	1    6050 5750
 	1    0    0    -1

Commit message: Works with KiCad V5.
Parts:
- C10, C11, C12, C13, C14, C8, C9: symbol C -> device:C
- U5: symbol SDRAM -> CAT-rescue:SDRAM
Changed lines of the file:
@@
-EESchema Schematic File Version 2
-LIBS:CAT-rescue
-LIBS:power
-LIBS:device
-LIBS:transistors
-LIBS:conn
-LIBS:linear
-LIBS:regul
-LIBS:74xx
-LIBS:cmos4000
-LIBS:adc-dac
-LIBS:memory
-LIBS:xilinx
-LIBS:microcontrollers
-LIBS:dsp
-LIBS:microchip
-LIBS:analog_switches
-LIBS:motorola
-LIBS:texas
-LIBS:intel
-LIBS:audio
-LIBS:interface
-LIBS:digital-audio
-LIBS:philips
-LIBS:display
-LIBS:cypress
-LIBS:siliconi
-LIBS:opto
-LIBS:atmel
-LIBS:contrib
-LIBS:valves
-LIBS:xess
-LIBS:Cypress_PSoC
-LIBS:Cypress_cy8c5xlp
-LIBS:Lattice_iCE_FPGA
-LIBS:xilinx7
-LIBS:xilinx6v
-LIBS:xilinx6s
-LIBS:xula
-LIBS:espressif-xess
+EESchema Schematic File Version 4
 LIBS:CAT-cache
 EELAYER 26 0
@@
 $EndDescr
 $Comp
-L SDRAM U5
+L CAT-rescue:SDRAM U5
 U 1 1 55E88707
 P 5500 2500
@@
 $EndComp
 $Comp
-L C C12
+L device:C C12
 U 1 1 55E9F330
 P 6350 5750
@@
 $EndComp
 $Comp
-L C C13
+L device:C C13
 U 1 1 55E9F363
 P 6650 5750
@@
 $EndComp
 $Comp
-L C C14
+L device:C C14
 U 1 1 55E9F939
 P 6950 5750
@@
 $EndComp
 $Comp
-L C C8
+L device:C C8
 U 1 1 55E9FAF7
 P 5150 5750
@@
 $EndComp
 $Comp
-L C C9
+L device:C C9
 U 1 1 55E9FAFD
 P 5450 5750
@@
 $EndComp
 $Comp
-L C C10
+L device:C C10
 U 1 1 55E9FB07
 P 5750 5750
@@
 $EndComp
 $Comp
-L C C11
+L device:C C11
 U 1 1 55E9FB0D
 P 6050 5750
