File: pcb/CAT-skidl.kicad_pcb (KiCad board)
At the start: 2 copper layers, 65 x 56 mm, 75 parts, among them J1 RPi_GPIO, J2 Conn_01x03, J3 Conn_01x03, J4 Conn_02x10_Odd_Even, J5 HDMI-FEMALE, SW1 SW_Push, SW2 SW_DIP_x04, SW3 SW_Push, SW4 SW_Push, U1 iCE40-HX8K-CT256, U2 SPI_FLASH_SOIC8, U3 EEPROM_I2C, U4 SDRAM_16Mx16_VFBGA-54, X1 ASE-xxxMHz

Commit message: Changed mailto link.
Parts:
- removed GR4, GR5: Grove_Male, xesscorp/xess.pretty:GROVE_MALE
- moved RN10 159.3 mm to (7.49, 14.1)
- moved RN9 137.4 mm to (12.1, 27.9)
- moved R3 136.3 mm to (11.7, 9.09)
- moved C27 135.9 mm to (29.7, 26.7)
- moved RN2 133.0 mm to (34.8, 9.90)
- moved C22 132.1 mm to (22.8, 20.8)
- moved C21 130.8 mm to (20.4, 20.8)
- moved D2 130.2 mm to (43.2, 41.1), turned to 90 degrees
- moved RN7 124.6 mm to (18.8, 44.3), turned to 180 degrees
- moved RN8 122.8 mm to (7.87, 43.6)
- moved C17 119.7 mm to (37.3, 10.9)
- moved C18 118.2 mm to (37.3, 9.23)
- moved GR3 117.8 mm to (3.43, 13.7), turned to 90 degrees
- moved J2 116.5 mm to (41.4, 49.0)
- moved C23 114.4 mm to (25.2, 20.8)
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Connections:
- net +5V-Raspi renamed RASPI_GPIO1_5V
- net B$51 renamed B$81
- net SD1_ADDR2 renamed SD1_DATA15
- net SD1_DATA0 renamed SD1_ADDR8
- GR1 pad 1: PM1_BUS1 -> GR1-IO1
- GR1 pad 2: PM1_BUS3 -> GR1-IO2
- GR1 pad 3: N$5 -> +3.3V
- GR2 pad 1: PM2_BUS1 -> GR2-IO1
- GR2 pad 2: PM2_BUS3 -> GR2-IO2
- GR2 pad 3: N$6 -> +3.3V
- GR3 pad 1: GR1-IO1 -> GR3-IO1
- GR3 pad 2: GR1-IO2 -> GR3-IO2
